File: kicad/lab7Kicad/lab7Kicad.kicad_sch (KiCad schematic)
At the start: 27 parts, among them M2 Motor, SW1 SW_Push, U1 PIC32MX170F256B, U2 SN754410, U3 USB2Serial, U4 Quadrature_Encoder

Commit message: Complete part 1.1 and complete prelab submission
Parts:
- added D11: 1N4935, symbol me218_library:Diode
- added M1: Motor, symbol me218_library:Motor
- added R5: 10, symbol me218_library:Res1
Connections:
- net GND is gone; now on net +3.3V: C1.1, C2.2, C3.2, C4.1, C5.2, D3.2 (A), D5.2 (A), D7.2 (A), D8.2 (A), PRG1.3 (Vss), RV1.3, SW1.1, U1.19 (Vss), U1.27 (AVss), U1.8 (Vss), U2.12 (GND), U2.13 (GND), U2.4 (GND), U2.5 (GND), U3.4 (GND), U4.4 (GND)
- net +3.3V: now also U1.3 (RA1), R5.2
- net at U2.9 (EN3,4): no longer U1.25 (RB14)
- new net: D11.2 (A), M1.2 (-), R5.1
Other:
- note added: "1A - Toggle between 1 and 0 (Via RA2)"
- note added: "1Y from SN754410"
- note added: "5V"
- note added: "DIRECTION PIN INPUT"
- note added: "Measurement Circuit for Electrical Time Constant"
- note added: "Toggle between 1 and 0 For Time Constant measurement"
- company: (none) -> Stanford
- title: (none) -> Lab 7
